File: pcb/TMP.kicad_sch (KiCad schematic)
At the start: 37 parts, among them J1 Conn_01x02_Pin, J2 Conn_01x02_Pin, J3 Conn_01x02_Pin, J4 Conn_01x03_Socket, U1 LM358

Commit message: Fix vendor/vendorid at bom
Parts:
- C1: Hersteller HTL -> (none); Nummer 100142 -> (none); Vendor (none) -> HTL; VendorId (none) -> 100142
- C2: Hersteller HTL -> (none); Nummer 100128 -> (none); Vendor (none) -> HTL; VendorId (none) -> 100128
- D1: Hersteller HTL -> (none); Nummer 100459 -> (none); Vendor (none) -> HTL; VendorId (none) -> 100459
- D2: Hersteller HTL -> (none); Nummer 100458 -> (none); Vendor (none) -> HTL; VendorId (none) -> 100458
- F1: Hersteller HTL -> (none); Nummer 101639 -> (none); Vendor (none) -> HTL; VendorId (none) -> 101639
- H1, H2, H3, H4: Hersteller HTL -> (none); Nummer 101018, 101382 -> (none); Vendor (none) -> HTL; VendorId (none) -> 101018, 101382
- J1, J3, J4: Hersteller HTL -> (none); Nummer 101521 -> (none); Vendor (none) -> HTL; VendorId (none) -> 101521
- J2: Hersteller HTL -> (none); Nummer 103421 -> (none); Vendor (none) -> HTL; VendorId (none) -> 103421
- R1: Hersteller HTL -> (none); Nummer 103422 -> (none); Vendor (none) -> HTL; VendorId (none) -> 103422
- R10: Hersteller HTL -> (none); Nummer 102765 -> (none); Vendor (none) -> HTL; VendorId (none) -> 102765
- R11: Hersteller HTL -> (none); Nummer 102902 -> (none); Vendor (none) -> HTL; VendorId (none) -> 102902
- R2: Hersteller HTL -> (none); Nummer 102940 -> (none); Vendor (none) -> HTL; VendorId (none) -> 102940
- R4: Hersteller HTL -> (none); Nummer 102960 -> (none); Vendor (none) -> HTL; VendorId (none) -> 102960
- R5, R7: Hersteller HTL -> (none); Nummer 102951 -> (none); Vendor (none) -> HTL; VendorId (none) -> 102951
- R6: Hersteller HTL -> (none); Nummer 102977 -> (none); Vendor (none) -> HTL; VendorId (none) -> 102977
- R8, R9: Hersteller HTL -> (none); Nummer 102938 -> (none); Vendor (none) -> HTL; VendorId (none) -> 102938
- RV1: Hersteller HTL -> (none); Nummer 103423 -> (none); Vendor (none) -> HTL; VendorId (none) -> 103423
- RV2, RV4: Hersteller HTL -> (none); Nummer 103424 -> (none); Vendor (none) -> HTL; VendorId (none) -> 103424
- RV3: Hersteller HTL -> (none); Nummer 100424 -> (none); Vendor (none) -> HTL; VendorId (none) -> 100424
- U1: Hersteller HTL -> (none); Nummer 100327 -> (none); Vendor (none) -> HTL; VendorId (none) -> 100327
