File: pcb/TMP.kicad_sch (KiCad schematic)
At the start: 37 parts, among them J1 Conn_01x02_Pin, J2 Conn_01x02_Pin, J3 Conn_01x02_Pin, J4 Conn_01x03_Socket, U1 LM358

Commit message: Update to KiCAD 9
Parts:
- added FID4: QR, Images:QR_0x007e, symbol Mechanical:Fiducial
- FID1, FID2, FID3: now left out of the parts list
Other:
- note added: "KTY81/210"
- moved on the sheet: FID1, FID2, FID3, H1, H2, H3, H4

Commit message: Rename/Add/Remove bom fields
Parts:
- C1: HTL (none) -> 100142; Vendor HTL -> (none); VendorId 100142 -> (none)
- C2: HTL (none) -> 100128; Vendor HTL -> (none); VendorId 100128 -> (none)
- D1: HTL (none) -> 100459; Vendor HTL -> (none); VendorId 100459 -> (none)
- D2: HTL (none) -> 100458; Vendor HTL -> (none); VendorId 100458 -> (none)
- F1: HTL (none) -> 101639; Vendor HTL -> (none); VendorId 101639 -> (none)
- H1, H2, H3, H4: HTL (none) -> 101018, 101382; Vendor HTL -> (none); VendorId 101018, 101382 -> (none)
- J1, J3, J4: HTL (none) -> 101521; Vendor HTL -> (none); VendorId 101521 -> (none)
- J2: HTL (none) -> 103421; Vendor HTL -> (none); VendorId 103421 -> (none)
- R1: HTL (none) -> 103422; Vendor HTL -> (none); VendorId 103422 -> (none)
- R10: HTL (none) -> 102765; Vendor HTL -> (none); VendorId 102765 -> (none)
- R11: HTL (none) -> 102902; Vendor HTL -> (none); VendorId 102902 -> (none)
- R2: HTL (none) -> 102940; Vendor HTL -> (none); VendorId 102940 -> (none)
- R4: HTL (none) -> 102960; Vendor HTL -> (none); VendorId 102960 -> (none)
- R5, R7: HTL (none) -> 102951; Vendor HTL -> (none); VendorId 102951 -> (none)
- R6: HTL (none) -> 102977; Vendor HTL -> (none); VendorId 102977 -> (none)
- R8, R9: HTL (none) -> 102938; Vendor HTL -> (none); VendorId 102938 -> (none)
- RV1: HTL (none) -> 103423; Vendor HTL -> (none); VendorId 103423 -> (none)
- RV2, RV4: HTL (none) -> 103424; Vendor HTL -> (none); VendorId 103424 -> (none)
- RV3: HTL (none) -> 100424; Vendor HTL -> (none); VendorId 100424 -> (none)
- TP1, TP2, TP3, TP4, TP5: now left out of the parts list
- U1: HTL (none) -> 100327; Vendor HTL -> (none); VendorId 100327 -> (none)

Commit message: Rename fiducial to bin
Parts:
- FID2: value Waste -> BIN
Changed lines of the file:
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@@
 			)
 		)
-		(property "Value" "Waste"
+		(property "Value" "BIN"
 			(at 232.41 146.05 0)
 			(effects
